Commit message: rightbot config pkg changes

File: rightbot_config_pkg/description/ros2_control/rrbot_modular_actuators.ros2_control_example.xacro (robot description, xacro)
@@ -2,4 +2,28 @@
 <robot xmlns:xacro="http://www.ros.org/wiki/xacro">
   <xacro:macro name="rrbot_modular_actuators" params="name prefix slowdown:=2.0">
+    <ros2_control name="RRBotModularJoint1" type="actuator">
+      <hardware>
+        <plugin>harmonic_motor_actuator</plugin>
+        <param name="example_param_hw_start_duration_sec">0</param>
+        <param name="example_param_hw_stop_duration_sec">3.0</param>
+        <param name="example_param_hw_slowdown">100</param>
+      </hardware>
+      <joint name="${prefix}joint1">
+        <command_interface name="position">
+          <param name="min">-100</param>
+          <param name="max">100</param>
+        </command_interface>
+        <command_interface name="max_velocity"/>
+        <command_interface name="acceleration"/>
+        <state_interface name="position"/>
+        <state_interface name="velocity"/>
+        <state_interface name="status"/>
+        <state_interface name="error_code"/>
+        <state_interface name="node_guard_error"/>
+        <param name="can_id">16</param>
+        <param name="axis">1</param>
+        <param name="path">"/home/rightbot/test_ws/src/ros2_control/rightbot_hardware_interface_pkgs/src/config/config.json"</param>
+      </joint>
+    </ros2_control>
     <ros2_control name="RRBotModularJoint2" type="actuator">
       <hardware>

File: rightbot_config_pkg/description/urdf/rrbot_modular_actuators.urdf.xacro (robot description, xacro)
@@ -10,9 +10,9 @@
   <xacro:arg name="slowdown" default="2.0" />
   <!-- Import RRBot macro -->
-  <xacro:include filename="$(find ros2_control_demo_example_6)/urdf/rrbot_description.urdf.xacro" />
+  <xacro:include filename="$(find rightbot_config_pkg)/urdf/rrbot_description.urdf.xacro" />
   <!-- Import Rviz colors -->
-  <xacro:include filename="$(find ros2_control_demo_example_6)/urdf/rrbot.materials.xacro" />
+  <xacro:include filename="$(find rightbot_config_pkg)/urdf/rrbot.materials.xacro" />
   <!-- Import RRBot ros2_control description -->
-  <xacro:include filename="$(find ros2_control_demo_example_6)/ros2_control/rrbot_modular_actuators.ros2_control.xacro" />
+  <xacro:include filename="$(find rightbot_config_pkg)/ros2_control/rrbot_modular_actuators.ros2_control.xacro" />
   <!-- Used for fixing robot -->
   <link name="world"/>
