Commit message: vertical gantry working

File: rightbot_config_pkg/description/ros2_control/rrbot_modular_actuators.ros2_control.xacro (robot description, xacro)
@@ -2,5 +2,5 @@
 <robot xmlns:xacro="http://www.ros.org/wiki/xacro">
   <xacro:macro name="rrbot_modular_actuators" params="name prefix slowdown:=2.0">
-    <ros2_control name="RRBotModularJoint2" type="actuator">
+    <ros2_control name="RRBotModularJoint1" type="actuator">
       <hardware>
         <plugin>motor_actuator</plugin>
@@ -9,5 +9,5 @@
         <param name="example_param_hw_slowdown">100</param>
       </hardware>
-      <joint name="${prefix}joint2">
+      <joint name="${prefix}joint1">
         <command_interface name="position">
           <param name="min">-100</param>
@@ -24,11 +24,14 @@
         <state_interface name="latched_fault"/>
         <state_interface name="node_guard_error"/>
-        <param name="can_id">13</param>
+        <param name="can_id">14</param>
         <param name="axis">1</param>
         <param name="path">"/home/rightbot/test_ws/src/ros2_control/rightbot_hardware_interface_pkgs/src/config/config.json"</param>
-        <param name="homing">"active"</param>
+        <param name="homing">1</param>
         <param name="homing_velocity">50</param>
         <param name="homing_acceleration">10</param>
-        <param name="homing_position">2000</param>
+        <param name="homing_position">0.951</param>
+        <param name="total_travel_distance">0.951</param>
+        <param name="motor_gear_ratio">7.5</param>
+        <param name="travel_per_revolution">0.314</param>
       </joint>
     </ros2_control>

File: rightbot_config_pkg/description/ros2_control/rrbot_modular_actuators.ros2_control_final_example.xacro (robot description, xacro)
@@ -51,8 +51,11 @@
         <param name="axis">1</param>
         <param name="path">"/home/rightbot/test_ws/src/ros2_control/rightbot_hardware_interface_pkgs/src/config/config.json"</param>
-        <param name="homing">"active"</param>
+        <param name="homing">1</param>
         <param name="homing_velocity">50</param>
         <param name="homing_acceleration">10</param>
-        <param name="homing_position">2000</param>
+        <param name="homing_position">0.9</param>
+        <param name="total_travel_distance">0.9</param>
+        <param name="motor_gear_ratio">7.5</param>
+        <param name="travel_per_revolution">0.314</param>
       </joint>
     </ros2_control>

Commit message: 2 gantry motor working

File: rightbot_config_pkg/description/ros2_control/rrbot_modular_actuators.ros2_control.xacro (robot description, xacro)
@@ -39,4 +39,41 @@
       </joint>
     </ros2_control>
+     <ros2_control name="RRBotModularJoint2" type="actuator">
+      <hardware>
+        <plugin>motor_actuator</plugin>
+        <param name="example_param_hw_start_duration_sec">0</param>
+        <param name="example_param_hw_stop_duration_sec">3.0</param>
+        <param name="example_param_hw_slowdown">100</param>
+      </hardware>
+      <joint name="${prefix}joint2">
+        <command_interface name="position">
+          <param name="min">-100</param>
+          <param name="max">100</param>
+        </command_interface>
+        <command_interface name="max_velocity"/>
+        <command_interface name="acceleration"/>
+        <state_interface name="position"/>
+        <state_interface name="velocity"/>
+        <state_interface name="status"/>
+        <state_interface name="battery_voltage"/>
+        <state_interface name="input_states"/>
+        <state_interface name="manufacturer_register"/>
+        <state_interface name="latched_fault"/>
+        <state_interface name="node_guard_error"/>
+        <param name="can_id">22</param>
+        <param name="axis">1</param>
+        <param name="path">"/home/rightbot/test_ws/src/ros2_control/rightbot_hardware_interface_pkgs/src/config/config.json"</param>
+        <param name="homing">1</param>
+        <param name="homing_at_zero">0</param>
+        <param name="homing_velocity">50</param>
+        <param name="homing_acceleration">10</param>
+        <param name="homing_position">0.951</param>
+        <param name="total_travel_distance">0.951</param>
+        <param name="motor_gear_ratio">7.5</param>
+        <param name="travel_per_revolution">0.314</param>
+        <param name="default_max_velocity">50.0</param>
+        <param name="default_max_accleration">10.0</param>
+      </joint>
+    </ros2_control>
   </xacro:macro>
 </robot>

File: rightbot_config_pkg/description/ros2_control/rrbot_modular_actuators.ros2_control_example.xacro (robot description, xacro)
@@ -57,4 +57,41 @@
       </joint>
     </ros2_control>
+     <ros2_control name="RRBotModularJoint1" type="actuator">
+      <hardware>
+        <plugin>motor_actuator</plugin>
+        <param name="example_param_hw_start_duration_sec">0</param>
+        <param name="example_param_hw_stop_duration_sec">3.0</param>
+        <param name="example_param_hw_slowdown">100</param>
+      </hardware>
+      <joint name="${prefix}joint1">
+        <command_interface name="position">
+          <param name="min">-100</param>
+          <param name="max">100</param>
+        </command_interface>
+        <command_interface name="max_velocity"/>
+        <command_interface name="acceleration"/>
+        <state_interface name="position"/>
+        <state_interface name="velocity"/>
+        <state_interface name="status"/>
+        <state_interface name="battery_voltage"/>
+        <state_interface name="input_states"/>
+        <state_interface name="manufacturer_register"/>
+        <state_interface name="latched_fault"/>
+        <state_interface name="node_guard_error"/>
+        <param name="can_id">16</param>
+        <param name="axis">1</param>
+        <param name="path">"/home/rightbot/test_ws/src/ros2_control/rightbot_hardware_interface_pkgs/src/config/config.json"</param>
+        <param name="homing">1</param>
+        <param name="homing_at_zero">1</param>
+        <param name="homing_velocity">50</param>
+        <param name="homing_acceleration">10</param>
+        <param name="homing_position">-0.747</param>
+        <param name="total_travel_distance">0.747</param>
+        <param name="motor_gear_ratio">1</param>
+        <param name="travel_per_revolution">0.032</param>
+        <param name="default_max_velocity">50.0</param>
+        <param name="default_max_accleration">10.0</param>
+      </joint>
+    </ros2_control>
   </xacro:macro>
 </robot>

Commit message: spawing all sherlock actuators

File: rightbot_config_pkg/description/ros2_control/rrbot_modular_actuators.ros2_control.xacro (robot description, xacro)
@@ -2,5 +2,79 @@
 <robot xmlns:xacro="http://www.ros.org/wiki/xacro">
   <xacro:macro name="rrbot_modular_actuators" params="name prefix slowdown:=2.0">
-    <ros2_control name="SherlockJoint1" type="actuator">
+     <ros2_control name="TruckUnloading_h_gantry_joint" type="actuator">
+      <hardware>
+        <plugin>motor_actuator</plugin>
+        <param name="example_param_hw_start_duration_sec">0</param>
+        <param name="example_param_hw_stop_duration_sec">3.0</param>
+        <param name="example_param_hw_slowdown">100</param>
+      </hardware>
+      <joint name="h_gantry_joint">
+        <command_interface name="position">
+          <param name="min">-100</param>
+          <param name="max">100</param>
+        </command_interface>
+        <command_interface name="max_velocity"/>
+        <command_interface name="acceleration"/>
+        <state_interface name="position"/>
+        <state_interface name="velocity"/>
+        <state_interface name="status"/>
+        <state_interface name="battery_voltage"/>
+        <state_interface name="input_states"/>
+        <state_interface name="manufacturer_register"/>
+        <state_interface name="latched_fault"/>
+        <state_interface name="node_guard_error"/>
+        <param name="can_id">16</param>
+        <param name="axis">1</param>
+        <param name="path">"/home/rightbot/test_ws/src/ros2_control/rightbot_hardware_interface_pkgs/src/config/config.json"</param>
+        <param name="homing">1</param>
+        <param name="homing_at_zero">1</param>
+        <param name="homing_velocity">50</param>
+        <param name="homing_acceleration">10</param>
+        <param name="homing_position">-0.747</param>
+        <param name="total_travel_distance">0.747</param>
+        <param name="motor_gear_ratio">1</param>
+        <param name="travel_per_revolution">0.032</param>
+        <param name="default_max_velocity">50.0</param>
+        <param name="default_max_accleration">10.0</param>
+      </joint>
+    </ros2_control>
+     <ros2_control name="TruckUnloading_v_gantry_joint" type="actuator">
+      <hardware>
+        <plugin>motor_actuator</plugin>
+        <param name="example_param_hw_start_duration_sec">0</param>
+        <param name="example_param_hw_stop_duration_sec">3.0</param>
+        <param name="example_param_hw_slowdown">100</param>
+      </hardware>
+      <joint name="v_gantry_joint">
+        <command_interface name="position">
+          <param name="min">-100</param>
+          <param name="max">100</param>
+        </command_interface>
+        <command_interface name="max_velocity"/>
+        <command_interface name="acceleration"/>
+        <state_interface name="position"/>
+        <state_interface name="velocity"/>
+        <state_interface name="status"/>
+        <state_interface name="battery_voltage"/>
+        <state_interface name="input_states"/>
+        <state_interface name="manufacturer_register"/>
+        <state_interface name="latched_fault"/>
+        <state_interface name="node_guard_error"/>
+        <param name="can_id">22</param>
+        <param name="axis">1</param>
+        <param name="path">"/home/rightbot/test_ws/src/ros2_control/rightbot_hardware_interface_pkgs/src/config/config.json"</param>
+        <param name="homing">1</param>
+        <param name="homing_at_zero">0</param>
+        <param name="homing_velocity">50</param>
+        <param name="homing_acceleration">10</param>
+        <param name="homing_position">0.951</param>
+        <param name="total_travel_distance">0.951</param>
+        <param name="motor_gear_ratio">7.5</param>
+        <param name="travel_per_revolution">0.314</param>
+        <param name="default_max_velocity">50.0</param>
+        <param name="default_max_accleration">10.0</param>
+      </joint>
+    </ros2_control>
+    <ros2_control name="TruckUnloading_base_rotation_joint" type="actuator">
       <hardware>
         <plugin>harmonic_motor_actuator</plugin>
@@ -22,4 +96,108 @@
         <state_interface name="node_guard_error"/>
         <param name="can_id">17</param>
+        <param name="axis">1</param>
+        <param name="path">"/home/rightbot/test_ws/src/ros2_control/rightbot_hardware_interface_pkgs/src/config/config.json"</param>
+        <param name="default_max_velocity">2</param>
+        <param name="default_max_accleration">1</param>
+      </joint>
+    </ros2_control>
+     <ros2_control name="TruckUnloading_elbow_rotation_joint" type="actuator">
+      <hardware>
+        <plugin>harmonic_motor_actuator</plugin>
+        <param name="example_param_hw_start_duration_sec">0</param>
+        <param name="example_param_hw_stop_duration_sec">3.0</param>
+        <param name="example_param_hw_slowdown">100</param>
+      </hardware>
+      <joint name="elbow_rotation_joint">
+        <command_interface name="position">
+          <param name="min">-100</param>
+          <param name="max">100</param>
+        </command_interface>
+        <command_interface name="max_velocity"/>
+        <command_interface name="acceleration"/>
+        <state_interface name="position"/>
+        <state_interface name="velocity"/>
+        <state_interface name="status"/>
+        <state_interface name="error_code"/>
+        <state_interface name="node_guard_error"/>
+        <param name="can_id">18</param>
+        <param name="axis">1</param>
+        <param name="path">"/home/rightbot/test_ws/src/ros2_control/rightbot_hardware_interface_pkgs/src/config/config.json"</param>
+        <param name="default_max_velocity">2</param>
+        <param name="default_max_accleration">1</param>
+      </joint>
+    </ros2_control>
+     <ros2_control name="TruckUnloading_wrist_rotation_joint" type="actuator">
+      <hardware>
+        <plugin>harmonic_motor_actuator</plugin>
+        <param name="example_param_hw_start_duration_sec">0</param>
+        <param name="example_param_hw_stop_duration_sec">3.0</param>
+        <param name="example_param_hw_slowdown">100</param>
+      </hardware>
+      <joint name="wrist_rotation_joint">
+        <command_interface name="position">
+          <param name="min">-100</param>
+          <param name="max">100</param>
+        </command_interface>
+        <command_interface name="max_velocity"/>
+        <command_interface name="acceleration"/>
+        <state_interface name="position"/>
+        <state_interface name="velocity"/>
+        <state_interface name="status"/>
+        <state_interface name="error_code"/>
+        <state_interface name="node_guard_error"/>
+        <param name="can_id">19</param>
+        <param name="axis">1</param>
+        <param name="path">"/home/rightbot/test_ws/src/ros2_control/rightbot_hardware_interface_pkgs/src/config/config.json"</param>
+        <param name="default_max_velocity">2</param>
+        <param name="default_max_accleration">1</param>
+      </joint>
+    </ros2_control>
+     <ros2_control name="TruckUnloading_rotation1_joint" type="actuator">
+      <hardware>
+        <plugin>harmonic_motor_actuator</plugin>
+        <param name="example_param_hw_start_duration_sec">0</param>
+        <param name="example_param_hw_stop_duration_sec">3.0</param>
+        <param name="example_param_hw_slowdown">100</param>
+      </hardware>
+      <joint name="rotation1_joint">
+        <command_interface name="position">
+          <param name="min">-100</param>
+          <param name="max">100</param>
+        </command_interface>
+        <command_interface name="max_velocity"/>
+        <command_interface name="acceleration"/>
+        <state_interface name="position"/>
+        <state_interface name="velocity"/>
+        <state_interface name="status"/>
+        <state_interface name="error_code"/>
+        <state_interface name="node_guard_error"/>
+        <param name="can_id">20</param>
+        <param name="axis">1</param>
+        <param name="path">"/home/rightbot/test_ws/src/ros2_control/rightbot_hardware_interface_pkgs/src/config/config.json"</param>
+        <param name="default_max_velocity">2</param>
+        <param name="default_max_accleration">1</param>
+      </joint>
+    </ros2_control>
+     <ros2_control name="TruckUnloading_rotation2_joint" type="actuator">
+      <hardware>
+        <plugin>harmonic_motor_actuator</plugin>
+        <param name="example_param_hw_start_duration_sec">0</param>
+        <param name="example_param_hw_stop_duration_sec">3.0</param>
+        <param name="example_param_hw_slowdown">100</param>
+      </hardware>
+      <joint name="rotation2_joint">
+        <command_interface name="position">
+          <param name="min">-100</param>
+          <param name="max">100</param>
+        </command_interface>
+        <command_interface name="max_velocity"/>
+        <command_interface name="acceleration"/>
+        <state_interface name="position"/>
+        <state_interface name="velocity"/>
+        <state_interface name="status"/>
+        <state_interface name="error_code"/>
+        <state_interface name="node_guard_error"/>
+        <param name="can_id">21</param>
         <param name="axis">1</param>
         <param name="path">"/home/rightbot/test_ws/src/ros2_control/rightbot_hardware_interface_pkgs/src/config/config.json"</param>
