Commit message: working

File: rightbot_config_pkg/description/ros2_control/rightbot_sherlock.ros2_control_old.xacro (robot description, xacro)
@@ -14,5 +14,5 @@
           <param name="max">100</param>
         </command_interface>
-        <command_interface name="velocity"/>
+        <command_interface name="max_velocity"/>
         <command_interface name="acceleration"/>
         <state_interface name="position"/>
@@ -24,5 +24,4 @@
         <state_interface name="latched_fault"/>
         <state_interface name="node_guard_error"/>
-        <state_interface name="actual_motor_current"/>
         <param name="can_id">16</param>
         <param name="axis">1</param>
@@ -52,5 +51,5 @@
           <param name="max">100</param>
         </command_interface>
-        <command_interface name="velocity"/>
+        <command_interface name="max_velocity"/>
         <command_interface name="acceleration"/>
         <state_interface name="position"/>
@@ -62,5 +61,4 @@
         <state_interface name="latched_fault"/>
         <state_interface name="node_guard_error"/>
-        <state_interface name="actual_motor_current"/>
         <param name="can_id">22</param>
         <param name="axis">1</param>
@@ -74,5 +72,5 @@
         <param name="motor_gear_ratio">7.5</param>
         <param name="travel_per_revolution">0.314</param>
-        <param name="default_max_velocity">80.0</param>
+        <param name="default_max_velocity">50.0</param>
         <param name="default_max_accleration">10.0</param>
       </joint>
@@ -90,17 +88,16 @@
           <param name="max">100</param>
         </command_interface>
-        <command_interface name="velocity"/>
-        <command_interface name="acceleration"/>
-        <state_interface name="position"/>
-        <state_interface name="velocity"/>
-        <state_interface name="status"/>
-        <state_interface name="error_code"/>
-        <state_interface name="node_guard_error"/>
-        <state_interface name="actual_motor_current"/>
+        <command_interface name="max_velocity"/>
+        <command_interface name="acceleration"/>
+        <state_interface name="position"/>
+        <state_interface name="velocity"/>
+        <state_interface name="status"/>
+        <state_interface name="error_code"/>
+        <state_interface name="node_guard_error"/>
         <param name="can_id">17</param>
-        <param name="axis">1</param>
-        <param name="path">"/home/rightbot/test_ws/src/ros2_control/rightbot_hardware_interface_pkgs/src/config/config.json"</param>
-        <param name="default_max_velocity">2</param>
-        <param name="default_max_accleration">0.5</param>
+        <param name="axis">-1</param>
+        <param name="path">"/home/rightbot/test_ws/src/ros2_control/rightbot_hardware_interface_pkgs/src/config/config.json"</param>
+        <param name="default_max_velocity">2</param>
+        <param name="default_max_accleration">1</param>
       </joint>
     </ros2_control>
@@ -117,17 +114,16 @@
           <param name="max">100</param>
         </command_interface>
-        <command_interface name="velocity"/>
-        <command_interface name="acceleration"/>
-        <state_interface name="position"/>
-        <state_interface name="velocity"/>
-        <state_interface name="status"/>
-        <state_interface name="error_code"/>
-        <state_interface name="node_guard_error"/>
-        <state_interface name="actual_motor_current"/>
+        <command_interface name="max_velocity"/>
+        <command_interface name="acceleration"/>
+        <state_interface name="position"/>
+        <state_interface name="velocity"/>
+        <state_interface name="status"/>
+        <state_interface name="error_code"/>
+        <state_interface name="node_guard_error"/>
         <param name="can_id">18</param>
         <param name="axis">-1</param>
         <param name="path">"/home/rightbot/test_ws/src/ros2_control/rightbot_hardware_interface_pkgs/src/config/config.json"</param>
         <param name="default_max_velocity">2</param>
-        <param name="default_max_accleration">0.5</param>
+        <param name="default_max_accleration">1</param>
       </joint>
     </ros2_control>
@@ -144,17 +140,16 @@
           <param name="max">100</param>
         </command_interface>
-        <command_interface name="velocity"/>
-        <command_interface name="acceleration"/>
-        <state_interface name="position"/>
-        <state_interface name="velocity"/>
-        <state_interface name="status"/>
-        <state_interface name="error_code"/>
-        <state_interface name="node_guard_error"/>
-        <state_interface name="actual_motor_current"/>
+        <command_interface name="max_velocity"/>
+        <command_interface name="acceleration"/>
+        <state_interface name="position"/>
+        <state_interface name="velocity"/>
+        <state_interface name="status"/>
+        <state_interface name="error_code"/>
+        <state_interface name="node_guard_error"/>
         <param name="can_id">19</param>
         <param name="axis">-1</param>
         <param name="path">"/home/rightbot/test_ws/src/ros2_control/rightbot_hardware_interface_pkgs/src/config/config.json"</param>
-        <param name="default_max_velocity">4</param>
-        <param name="default_max_accleration">0.5</param>
+        <param name="default_max_velocity">2</param>
+        <param name="default_max_accleration">1</param>
       </joint>
     </ros2_control>
@@ -171,17 +166,16 @@
           <param name="max">100</param>
         </command_interface>
-        <command_interface name="velocity"/>
-        <command_interface name="acceleration"/>
-        <state_interface name="position"/>
-        <state_interface name="velocity"/>
-        <state_interface name="status"/>
-        <state_interface name="error_code"/>
-        <state_interface name="node_guard_error"/>
-        <state_interface name="actual_motor_current"/>
+        <command_interface name="max_velocity"/>
+        <command_interface name="acceleration"/>
+        <state_interface name="position"/>
+        <state_interface name="velocity"/>
+        <state_interface name="status"/>
+        <state_interface name="error_code"/>
+        <state_interface name="node_guard_error"/>
         <param name="can_id">20</param>
         <param name="axis">-1</param>
         <param name="path">"/home/rightbot/test_ws/src/ros2_control/rightbot_hardware_interface_pkgs/src/config/config.json"</param>
-        <param name="default_max_velocity">4</param>
-        <param name="default_max_accleration">0.5</param>
+        <param name="default_max_velocity">2</param>
+        <param name="default_max_accleration">1</param>
       </joint>
     </ros2_control>
@@ -198,17 +192,16 @@
           <param name="max">100</param>
         </command_interface>
-        <command_interface name="velocity"/>
-        <command_interface name="acceleration"/>
-        <state_interface name="position"/>
-        <state_interface name="velocity"/>
-        <state_interface name="status"/>
-        <state_interface name="error_code"/>
-        <state_interface name="node_guard_error"/>
-        <state_interface name="actual_motor_current"/>
+        <command_interface name="max_velocity"/>
+        <command_interface name="acceleration"/>
+        <state_interface name="position"/>
+        <state_interface name="velocity"/>
+        <state_interface name="status"/>
+        <state_interface name="error_code"/>
+        <state_interface name="node_guard_error"/>
         <param name="can_id">21</param>
         <param name="axis">-1</param>
         <param name="path">"/home/rightbot/test_ws/src/ros2_control/rightbot_hardware_interface_pkgs/src/config/config.json"</param>
-        <param name="default_max_velocity">4</param>
-        <param name="default_max_accleration">0.5</param>
+        <param name="default_max_velocity">2</param>
+        <param name="default_max_accleration">1</param>
       </joint>
     </ros2_control>

File: rightbot_config_pkg/description/ros2_control/rightbot_test.ros2_control.xacro (robot description, xacro)
@@ -40,5 +40,5 @@
       </joint>
     </ros2_control>
-    <!-- <ros2_control name="TruckUnloading_base_rotation_joint" type="actuator">
+    <ros2_control name="TruckUnloading_rotation1_joint" type="actuator">
       <hardware>
         <plugin>harmonic_motor_actuator</plugin>
@@ -47,10 +47,10 @@
         <param name="example_param_hw_slowdown">100</param>
       </hardware>
-      <joint name="base_rotation_joint">
+      <joint name="rotation1_joint">
         <command_interface name="position">
           <param name="min">-100</param>
           <param name="max">100</param>
         </command_interface>
-        <command_interface name="max_velocity"/>
+        <command_interface name="velocity"/>
         <command_interface name="acceleration"/>
         <state_interface name="position"/>
@@ -59,5 +59,6 @@
         <state_interface name="error_code"/>
         <state_interface name="node_guard_error"/>
-        <param name="can_id">17</param>
+        <state_interface name="actual_motor_current"/>
+        <param name="can_id">20</param>
         <param name="axis">-1</param>
         <param name="path">"/home/rightbot/test_ws/src/ros2_control/rightbot_hardware_interface_pkgs/src/config/config.json"</param>
@@ -65,5 +66,5 @@
         <param name="default_max_accleration">1</param>
       </joint>
-    </ros2_control> -->
+    </ros2_control>
   </xacro:macro>
 </robot>
