Commit message: rightbot config pkg files names changed

File: rightbot_config_pkg/description/ros2_control/rightbot_sherlock.ros2_control.xacro (robot description, xacro)
@@ -1,5 +1,5 @@
 <?xml version="1.0"?>
 <robot xmlns:xacro="http://www.ros.org/wiki/xacro">
-  <xacro:macro name="rrbot_modular_actuators" params="name prefix slowdown:=2.0">
+  <xacro:macro name="rightbot_sherlock" params="name prefix slowdown:=2.0">
      <ros2_control name="TruckUnloading_h_gantry_joint" type="actuator">
       <hardware>

File: rightbot_config_pkg/description/urdf/rightbot_sherlock.urdf.xacro (robot description, xacro)
@@ -14,5 +14,5 @@
   <xacro:include filename="$(find rightbot_config_pkg)/urdf/rrbot.materials.xacro" />
   <!-- Import RRBot ros2_control description -->
-  <xacro:include filename="$(find rightbot_config_pkg)/ros2_control/rrbot_modular_actuators.ros2_control.xacro" />
+  <xacro:include filename="$(find rightbot_config_pkg)/ros2_control/rightbot_sherlock.ros2_control.xacro" />
   <!-- Used for fixing robot -->
   <link name="world"/>
@@ -20,6 +20,6 @@
     <origin xyz="0 0 0" rpy="0 0 0" />
   </xacro:rrbot>
-  <xacro:rrbot_modular_actuators
-    name="RRBotModularJoint" prefix="$(arg prefix)"
+  <xacro:rightbot_sherlock
+    name="RightbotSherlock" prefix="$(arg prefix)"
     slowdown="$(arg slowdown)" />
 </robot>

Commit message: joint initialization sequence change

File: rightbot_config_pkg/description/ros2_control/rightbot_sherlock.ros2_control.xacro (robot description, xacro)
@@ -40,4 +40,31 @@
       </joint>
     </ros2_control> -->
+    <ros2_control name="TruckUnloading_base_rotation_joint" type="actuator">
+      <hardware>
+        <plugin>harmonic_motor_actuator</plugin>
+        <param name="example_param_hw_start_duration_sec">0</param>
+        <param name="example_param_hw_stop_duration_sec">3.0</param>
+        <param name="example_param_hw_slowdown">100</param>
+      </hardware>
+      <joint name="base_rotation_joint">
+        <command_interface name="position">
+          <param name="min">-100</param>
+          <param name="max">100</param>
+        </command_interface>
+        <command_interface name="velocity"/>
+        <command_interface name="acceleration"/>
+        <state_interface name="position"/>
+        <state_interface name="velocity"/>
+        <state_interface name="status"/>
+        <state_interface name="error_code"/>
+        <state_interface name="node_guard_error"/>
+        <state_interface name="actual_motor_current"/>
+        <param name="can_id">17</param>
+        <param name="axis">1</param>
+        <param name="path">"/home/rightbot/test_ws/src/ros2_control/rightbot_hardware_interface_pkgs/src/config/config.json"</param>
+        <param name="default_max_velocity">2</param>
+        <param name="default_max_accleration">0.5</param>
+      </joint>
+    </ros2_control>
      <ros2_control name="TruckUnloading_v_gantry_joint" type="actuator">
       <hardware>
@@ -78,31 +105,4 @@
       </joint>
     </ros2_control>
-    <ros2_control name="TruckUnloading_base_rotation_joint" type="actuator">
-      <hardware>
-        <plugin>harmonic_motor_actuator</plugin>
-        <param name="example_param_hw_start_duration_sec">0</param>
-        <param name="example_param_hw_stop_duration_sec">3.0</param>
-        <param name="example_param_hw_slowdown">100</param>
-      </hardware>
-      <joint name="base_rotation_joint">
-        <command_interface name="position">
-          <param name="min">-100</param>
-          <param name="max">100</param>
-        </command_interface>
-        <command_interface name="velocity"/>
-        <command_interface name="acceleration"/>
-        <state_interface name="position"/>
-        <state_interface name="velocity"/>
-        <state_interface name="status"/>
-        <state_interface name="error_code"/>
-        <state_interface name="node_guard_error"/>
-        <state_interface name="actual_motor_current"/>
-        <param name="can_id">17</param>
-        <param name="axis">1</param>
-        <param name="path">"/home/rightbot/test_ws/src/ros2_control/rightbot_hardware_interface_pkgs/src/config/config.json"</param>
-        <param name="default_max_velocity">2</param>
-        <param name="default_max_accleration">0.5</param>
-      </joint>
-    </ros2_control>
      <ros2_control name="TruckUnloading_elbow_rotation_joint" type="actuator">
       <hardware>

Commit message: underprogress

File: rightbot_config_pkg/description/ros2_control/rightbot_sherlock.ros2_control.xacro (robot description, xacro)
@@ -222,4 +222,38 @@
       </joint>
     </ros2_control>
+    <ros2_control name="TruckUnloading_camera_joint" type="actuator">
+      <hardware>
+        <plugin>motor_actuator</plugin>
+        <param name="example_param_hw_start_duration_sec">0</param>
+        <param name="example_param_hw_stop_duration_sec">3.0</param>
+        <param name="example_param_hw_slowdown">100</param>
+      </hardware>
+      <joint name="camera_joint">
+        <command_interface name="position">
+          <param name="min">-100</param>
+          <param name="max">100</param>
+        </command_interface>
+        <command_interface name="velocity"/>
+        <command_interface name="acceleration"/>
+        <command_interface name="control_state"/>
+        <command_interface name="gpio"/>
+        <state_interface name="position"/>
+        <state_interface name="velocity"/>
+        <state_interface name="status"/>
+        <state_interface name="battery_voltage"/>
+        <state_interface name="input_states"/>
+        <state_interface name="manufacturer_register"/>
+        <state_interface name="latched_fault"/>
+        <state_interface name="node_guard_error"/>
+        <state_interface name="effort"/>
+        <param name="can_id">23</param>
+        <param name="axis">1</param>
+        <param name="path">"/home/rightbot/test_ws/src/ros2_control/rightbot_hardware_interface_pkgs/src/config/config.json"</param>
+        <param name="homing">0</param>
+        <param name="motor_gear_ratio">7.5</param>
+        <param name="default_max_velocity">50.0</param>
+        <param name="default_max_accleration">10.0</param>
+      </joint>
+    </ros2_control>
   </xacro:macro>
 </robot>
