Commit message: recent ros2_control.xacro

File: rightbot_config_pkg/description/ros2_control/rightbot_sherlock.ros2_control.xacro (robot description, xacro)
@@ -2,5 +2,35 @@
 <robot xmlns:xacro="http://www.ros.org/wiki/xacro">
   <xacro:macro name="rightbot_sherlock" params="name prefix slowdown:=2.0">
-     <ros2_control name="TruckUnloading_h_gantry_joint" type="actuator">
+    <ros2_control name="${name}_TruckUnloading_elbow_rotation_joint" type="actuator">
+      <hardware>
+        <plugin>harmonic_motor_actuator</plugin>
+        <param name="example_param_hw_start_duration_sec">0</param>
+        <param name="example_param_hw_stop_duration_sec">3.0</param>
+        <param name="example_param_hw_slowdown">100</param>
+      </hardware>
+      <joint name="elbow_rotation_joint">
+        <command_interface name="position">
+          <param name="min">-100</param>
+          <param name="max">100</param>
+        </command_interface>
+        <command_interface name="velocity"/>
+        <command_interface name="acceleration"/>
+        <command_interface name="control_state"/>
+        <state_interface name="position"/>
+        <state_interface name="velocity"/>
+        <state_interface name="status"/>
+        <state_interface name="error_code"/>
+        <state_interface name="node_guard_error"/>
+        <state_interface name="effort"/>
+        <param name="can_id">18</param>
+        <param name="axis">1</param>
+        <param name="default_max_velocity">2</param>
+        <param name="default_max_accleration">0.5</param>
+        <param name="path">
+          "/home/rightbot/test_ws/src/ros2_control/rightbot_hardware_interface_pkgs/src/config/config.json"
+        </param>
+      </joint>
+    </ros2_control>
+    <ros2_control name="${name}_TruckUnloading_h_gantry_joint" type="actuator">
       <hardware>
         <plugin>motor_actuator</plugin>
@@ -28,47 +58,21 @@
         <state_interface name="effort"/>
         <param name="can_id">16</param>
-        <param name="axis">1</param>
-        <param name="path">"/home/rightbot/test_ws/src/ros2_control/rightbot_hardware_interface_pkgs/src/config/config.json"</param>
+        <param name="axis">-1</param>
+        <param name="path">
+          "/home/rightbot/test_ws/src/ros2_control/rightbot_hardware_interface_pkgs/src/config/config.json"
+        </param>
         <param name="homing">1</param>
         <param name="homing_at_zero">1</param>
         <param name="homing_velocity">50</param>
         <param name="homing_acceleration">10</param>
-        <param name="homing_position">-0.747</param>
-        <param name="total_travel_distance">0.747</param>
+        <param name="homing_position">0.709</param>
+        <param name="total_travel_distance">0.709</param>
         <param name="motor_gear_ratio">1</param>
         <param name="travel_per_revolution">0.032</param>
         <param name="default_max_velocity">50.0</param>
-        <param name="default_max_accleration">10.0</param>
-      </joint>
-    </ros2_control>
-    <ros2_control name="TruckUnloading_base_rotation_joint" type="actuator">
-      <hardware>
-        <plugin>harmonic_motor_actuator</plugin>
-        <param name="example_param_hw_start_duration_sec">0</param>
-        <param name="example_param_hw_stop_duration_sec">3.0</param>
-        <param name="example_param_hw_slowdown">100</param>
-      </hardware>
-      <joint name="base_rotation_joint">
-        <command_interface name="position">
-          <param name="min">-100</param>
-          <param name="max">100</param>
-        </command_interface>
-        <command_interface name="velocity"/>
-        <command_interface name="acceleration"/>
-        <command_interface name="control_state"/>
-        <state_interface name="position"/>
-        <state_interface name="velocity"/>
-        <state_interface name="status"/>
-        <state_interface name="error_code"/>
-        <state_interface name="node_guard_error"/>
-        <state_interface name="effort"/>
-        <param name="can_id">17</param>
-        <param name="axis">1</param>
-        <param name="path">"/home/rightbot/test_ws/src/ros2_control/rightbot_hardware_interface_pkgs/src/config/config.json"</param>
-        <param name="default_max_velocity">2</param>
-        <param name="default_max_accleration">0.5</param>
-      </joint>
-    </ros2_control>
-     <ros2_control name="TruckUnloading_v_gantry_joint" type="actuator">
+        <param name="default_max_accleration">25.0</param>
+      </joint>
+    </ros2_control>
+    <ros2_control name="${name}_TruckUnloading_v_gantry_joint" type="actuator">
       <hardware>
         <plugin>motor_actuator</plugin>
@@ -96,164 +100,140 @@
         <state_interface name="effort"/>
         <param name="can_id">22</param>
-        <param name="axis">1</param>
-        <param name="path">"/home/rightbot/test_ws/src/ros2_control/rightbot_hardware_interface_pkgs/src/config/config.json"</param>
+        <param name="axis">-1</param>
         <param name="homing">1</param>
         <param name="homing_at_zero">0</param>
         <param name="homing_velocity">50</param>
         <param name="homing_acceleration">10</param>
-        <param name="homing_position">0.951</param>
+        <param name="homing_position">-0.951</param>
         <param name="total_travel_distance">0.951</param>
         <param name="motor_gear_ratio">7.5</param>
         <param name="travel_per_revolution">0.314</param>
         <param name="default_max_velocity">80.0</param>
-        <param name="default_max_accleration">10.0</param>
-      </joint>
-    </ros2_control>
-     <ros2_control name="TruckUnloading_elbow_rotation_joint" type="actuator">
-      <hardware>
-        <plugin>harmonic_motor_actuator</plugin>
-        <param name="example_param_hw_start_duration_sec">0</param>
-        <param name="example_param_hw_stop_duration_sec">3.0</param>
-        <param name="example_param_hw_slowdown">100</param>
-      </hardware>
-      <joint name="elbow_rotation_joint">
-        <command_interface name="position">
-          <param name="min">-100</param>
-          <param name="max">100</param>
-        </command_interface>
-        <command_interface name="velocity"/>
-        <command_interface name="acceleration"/>
-        <command_interface name="control_state"/>
-        <state_interface name="position"/>
-        <state_interface name="velocity"/>
-        <state_interface name="status"/>
-        <state_interface name="error_code"/>
-        <state_interface name="node_guard_error"/>
-        <state_interface name="effort"/>
-        <param name="can_id">18</param>
-        <param name="axis">-1</param>
-        <param name="path">"/home/rightbot/test_ws/src/ros2_control/rightbot_hardware_interface_pkgs/src/config/config.json"</param>
-        <param name="default_max_velocity">2</param>
-        <param name="default_max_accleration">0.5</param>
-      </joint>
-    </ros2_control>
-     <ros2_control name="TruckUnloading_wrist_rotation_joint" type="actuator">
-      <hardware>
-        <plugin>harmonic_motor_actuator</plugin>
-        <param name="example_param_hw_start_duration_sec">0</param>
-        <param name="example_param_hw_stop_duration_sec">3.0</param>
-        <param name="example_param_hw_slowdown">100</param>
-      </hardware>
-      <joint name="wrist_rotation_joint">
-        <command_interface name="position">
-          <param name="min">-100</param>
-          <param name="max">100</param>
-        </command_interface>
-        <command_interface name="velocity"/>
-        <command_interface name="acceleration"/>
-        <command_interface name="control_state"/>
-        <state_interface name="position"/>
-        <state_interface name="velocity"/>
-        <state_interface name="status"/>
-        <state_interface name="error_code"/>
-        <state_interface name="node_guard_error"/>
-        <state_interface name="effort"/>
-        <param name="can_id">19</param>
-        <param name="axis">1</param>
-        <param name="path">"/home/rightbot/test_ws/src/ros2_control/rightbot_hardware_interface_pkgs/src/config/config.json"</param>
-        <param name="default_max_velocity">4</param>
-        <param name="default_max_accleration">0.5</param>
-      </joint>
-    </ros2_control>
-     <ros2_control name="TruckUnloading_rotation1_joint" type="actuator">
-      <hardware>
-        <plugin>harmonic_motor_actuator</plugin>
-        <param name="example_param_hw_start_duration_sec">0</param>
-        <param name="example_param_hw_stop_duration_sec">3.0</param>
-        <param name="example_param_hw_slowdown">100</param>
-      </hardware>
-      <joint name="rotation1_joint">
-        <command_interface name="position">
-          <param name="min">-100</param>
-          <param name="max">100</param>
-        </command_interface>
-        <command_interface name="velocity"/>
-        <command_interface name="acceleration"/>
-        <command_interface name="control_state"/>
-        <state_interface name="position"/>
-        <state_interface name="velocity"/>
-        <state_interface name="status"/>
-        <state_interface name="error_code"/>
-        <state_interface name="node_guard_error"/>
-        <state_interface name="effort"/>
-        <param name="can_id">20</param>
-        <param name="axis">-1</param>
-        <param name="path">"/home/rightbot/test_ws/src/ros2_control/rightbot_hardware_interface_pkgs/src/config/config.json"</param>
-        <param name="default_max_velocity">4</param>
-        <param name="default_max_accleration">0.5</param>
-      </joint>
-    </ros2_control>
-     <ros2_control name="TruckUnloading_rotation2_joint" type="actuator">
-      <hardware>
-        <plugin>harmonic_motor_actuator</plugin>
-        <param name="example_param_hw_start_duration_sec">0</param>
-        <param name="example_param_hw_stop_duration_sec">3.0</param>
-        <param name="example_param_hw_slowdown">100</param>
-      </hardware>
-      <joint name="rotation2_joint">
-        <command_interface name="position">
-          <param name="min">-100</param>
-          <param name="max">100</param>
-        </command_interface>
-        <command_interface name="velocity"/>
-        <command_interface name="acceleration"/>
-        <command_interface name="control_state"/>
-        <state_interface name="position"/>
-        <state_interface name="velocity"/>
-        <state_interface name="status"/>
-        <state_interface name="error_code"/>
-        <state_interface name="node_guard_error"/>
-        <state_interface name="effort"/>
-        <param name="can_id">21</param>
-        <param name="axis">-1</param>
-        <param name="path">"/home/rightbot/test_ws/src/ros2_control/rightbot_hardware_interface_pkgs/src/config/config.json"</param>
-        <param name="default_max_velocity">4</param>
-        <param name="default_max_accleration">0.5</param>
-      </joint>
-    </ros2_control>
-    <ros2_control name="TruckUnloading_camera_joint" type="actuator">
-      <hardware>
-        <plugin>motor_actuator</plugin>
-        <param name="example_param_hw_start_duration_sec">0</param>
-        <param name="example_param_hw_stop_duration_sec">3.0</param>
-        <param name="example_param_hw_slowdown">100</param>
-      </hardware>
-      <joint name="camera_joint">
-        <command_interface name="position">
-          <param name="min">-100</param>
-          <param name="max">100</param>
-        </command_interface>
-        <command_interface name="velocity"/>
-        <command_interface name="acceleration"/>
-        <command_interface name="control_state"/>
-        <command_interface name="gpio"/>
-        <state_interface name="position"/>
-        <state_interface name="velocity"/>
-        <state_interface name="status"/>
-        <state_interface name="battery_voltage"/>
-        <state_interface name="input_states"/>
-        <state_interface name="manufacturer_register"/>
-        <state_interface name="latched_fault"/>
-        <state_interface name="node_guard_error"/>
-        <state_interface name="effort"/>
-        <param name="can_id">23</param>
-        <param name="axis">1</param>
-        <param name="path">"/home/rightbot/test_ws/src/ros2_control/rightbot_hardware_interface_pkgs/src/config/config.json"</param>
-        <param name="homing">0</param>
-        <param name="motor_gear_ratio">7.5</param>
-        <param name="default_max_velocity">50.0</param>
-        <param name="default_max_accleration">10.0</param>
-      </joint>
-    </ros2_control>
+        <param name="default_max_accleration">25.0</param>
+        <param name="path">
+          "/home/rightbot/test_ws/src/ros2_control/rightbot_hardware_interface_pkgs/src/config/config.json"
+        </param>
+      </joint>
+    </ros2_control>
+    <ros2_control name="${name}_TruckUnloading_base_rotation_joint" type="actuator">
+      <hardware>
+          <plugin>harmonic_motor_actuator</plugin>
+          <param name="example_param_hw_start_duration_sec">0</param>
+          <param name="example_param_hw_stop_duration_sec">3.0</param>
+          <param name="example_param_hw_slowdown">100</param>
+      </hardware>
+      <joint name="base_rotation_joint">
+          <command_interface name="position">
+              <param name="min">-100</param>
+              <param name="max">100</param>
+          </command_interface>
+          <command_interface name="velocity"/>
+          <command_interface name="acceleration"/>
+          <command_interface name="control_state"/>
+          <state_interface name="position"/>
+          <state_interface name="velocity"/>
+          <state_interface name="status"/>
+          <state_interface name="error_code"/>
+          <state_interface name="node_guard_error"/>
+          <state_interface name="effort"/>
+          <param name="can_id">17</param>
+          <param name="axis">-1</param>
+          <param name="default_max_velocity">2</param>
+          <param name="default_max_accleration">0.5</param>
+          <param name="path">
+              "/home/rightbot/test_ws/src/ros2_control/rightbot_hardware_interface_pkgs/src/config/config.json"
+          </param>
+      </joint>
+    </ros2_control>
+        <ros2_control name="${name}_TruckUnloading_wrist_rotation_joint" type="actuator">
+            <hardware>
+                <plugin>harmonic_motor_actuator</plugin>
+                <param name="example_param_hw_start_duration_sec">0</param>
+                <param name="example_param_hw_stop_duration_sec">3.0</param>
+                <param name="example_param_hw_slowdown">100</param>
+            </hardware>
+            <joint name="wrist_rotation_joint">
+                <command_interface name="position">
+                    <param name="min">-100</param>
+                    <param name="max">100</param>
+                </command_interface>
+                <command_interface name="velocity"/>
+                <command_interface name="acceleration"/>
+                <command_interface name="control_state"/>
+                <state_interface name="position"/>
+                <state_interface name="velocity"/>
+                <state_interface name="status"/>
+                <state_interface name="error_code"/>
+                <state_interface name="node_guard_error"/>
+                <state_interface name="effort"/>
+                <param name="can_id">19</param>
+                <param name="axis">-1</param>
+                <param name="default_max_velocity">4</param>
+                <param name="default_max_accleration">0.5</param>
+                <param name="path">
+                    "/home/rightbot/test_ws/src/ros2_control/rightbot_hardware_interface_pkgs/src/config/config.json"
+                </param>
+            </joint>
+        </ros2_control>
+        <ros2_control name="${name}_TruckUnloading_rotation1_joint" type="actuator">
+            <hardware>
+                <plugin>harmonic_motor_actuator</plugin>
+                <param name="example_param_hw_start_duration_sec">0</param>
+                <param name="example_param_hw_stop_duration_sec">3.0</param>
+                <param name="example_param_hw_slowdown">100</param>
+            </hardware>
+            <joint name="rotation1_joint">
+                <command_interface name="position">
+                    <param name="min">-100</param>
+                    <param name="max">100</param>
+                </command_interface>
+                <command_interface name="velocity"/>
+                <command_interface name="acceleration"/>
+                <command_interface name="control_state"/>
+                <state_interface name="position"/>
+                <state_interface name="velocity"/>
+                <state_interface name="status"/>
+                <state_interface name="error_code"/>
+                <state_interface name="node_guard_error"/>
+                <state_interface name="effort"/>
+                <param name="can_id">20</param>
+                <param name="axis">1</param>
+                <param name="default_max_velocity">4</param>
+                <param name="default_max_accleration">0.5</param>
+                <param name="path">
+                    "/home/rightbot/test_ws/src/ros2_control/rightbot_hardware_interface_pkgs/src/config/config.json"
+                </param>
+            </joint>
+        </ros2_control>
+        <ros2_control name="${name}_TruckUnloading_rotation2_joint" type="actuator">
+            <hardware>
+                <plugin>harmonic_motor_actuator</plugin>
+                <param name="example_param_hw_start_duration_sec">0</param>
+                <param name="example_param_hw_stop_duration_sec">3.0</param>
+                <param name="example_param_hw_slowdown">100</param>
+            </hardware>
+            <joint name="rotation2_joint">
+                <command_interface name="position">
+                    <param name="min">-100</param>
+                    <param name="max">100</param>
+                </command_interface>
+                <command_interface name="velocity"/>
+                <command_interface name="acceleration"/>
+                <command_interface name="control_state"/>
+                <state_interface name="position"/>
+                <state_interface name="velocity"/>
+                <state_interface name="status"/>
+                <state_interface name="error_code"/>
+                <state_interface name="node_guard_error"/>
+                <state_interface name="effort"/>
+                <param name="can_id">21</param>
+                <param name="axis">-1</param>
+                <param name="default_max_velocity">4</param>
+                <param name="default_max_accleration">0.5</param>
+                <param name="path">
+                    "/home/rightbot/test_ws/src/ros2_control/rightbot_hardware_interface_pkgs/src/config/config.json"
+                </param>
+            </joint>
+        </ros2_control>
   </xacro:macro>
 </robot>
