Commit message: acceleration interface

File: rightbot_config_pkg/description/ros2_control/rightbot_test.ros2_control.xacro (robot description, xacro)
@@ -2,5 +2,5 @@
 <robot xmlns:xacro="http://www.ros.org/wiki/xacro">
   <xacro:macro name="rightbot_test" params="name prefix slowdown:=2.0">
-     <ros2_control name="TruckUnloading_h_gantry_joint" type="actuator">
+    <ros2_control name="TruckUnloading_v_gantry_joint" type="actuator">
       <hardware>
         <plugin>motor_actuator</plugin>
@@ -9,10 +9,10 @@
         <param name="example_param_hw_slowdown">100</param>
       </hardware>
-      <joint name="h_gantry_joint">
+      <joint name="v_gantry_joint">
         <command_interface name="position">
           <param name="min">-100</param>
           <param name="max">100</param>
         </command_interface>
-        <command_interface name="max_velocity"/>
+        <command_interface name="velocity"/>
         <command_interface name="acceleration"/>
         <state_interface name="position"/>
@@ -25,20 +25,20 @@
         <state_interface name="node_guard_error"/>
         <state_interface name="actual_motor_current"/>
-        <param name="can_id">16</param>
+        <param name="can_id">22</param>
         <param name="axis">1</param>
         <param name="path">"/home/rightbot/test_ws/src/ros2_control/rightbot_hardware_interface_pkgs/src/config/config.json"</param>
         <param name="homing">1</param>
-        <param name="homing_at_zero">1</param>
+        <param name="homing_at_zero">0</param>
         <param name="homing_velocity">50</param>
         <param name="homing_acceleration">10</param>
-        <param name="homing_position">0.0</param>
-        <param name="total_travel_distance">0.747</param>
+        <param name="homing_position">0.951</param>
+        <param name="total_travel_distance">0.951</param>
         <param name="motor_gear_ratio">7.5</param>
-        <param name="travel_per_revolution">0.032</param>
+        <param name="travel_per_revolution">0.314</param>
         <param name="default_max_velocity">50.0</param>
         <param name="default_max_accleration">10.0</param>
       </joint>
     </ros2_control>
-    <ros2_control name="TruckUnloading_base_rotation_joint" type="actuator">
+    <!-- <ros2_control name="TruckUnloading_base_rotation_joint" type="actuator">
       <hardware>
         <plugin>harmonic_motor_actuator</plugin>
@@ -65,5 +65,5 @@
         <param name="default_max_accleration">1</param>
       </joint>
-    </ros2_control>
+    </ros2_control> -->
   </xacro:macro>
 </robot>

Commit message: test config changes + rightbot_sherlock at 100Hz

File: rightbot_config_pkg/description/ros2_control/rightbot_test.ros2_control.xacro (robot description, xacro)
@@ -2,12 +2,12 @@
 <robot xmlns:xacro="http://www.ros.org/wiki/xacro">
   <xacro:macro name="rightbot_test" params="name prefix slowdown:=2.0">
-    <ros2_control name="TruckUnloading_v_gantry_joint" type="actuator">
+    <ros2_control name="TruckUnloading_base_rotation_joint" type="actuator">
       <hardware>
-        <plugin>motor_actuator</plugin>
+        <plugin>harmonic_motor_actuator</plugin>
         <param name="example_param_hw_start_duration_sec">0</param>
         <param name="example_param_hw_stop_duration_sec">3.0</param>
         <param name="example_param_hw_slowdown">100</param>
       </hardware>
-      <joint name="v_gantry_joint">
+      <joint name="base_rotation_joint">
         <command_interface name="position">
           <param name="min">-100</param>
@@ -19,26 +19,69 @@
         <state_interface name="velocity"/>
         <state_interface name="status"/>
-        <state_interface name="battery_voltage"/>
-        <state_interface name="input_states"/>
-        <state_interface name="manufacturer_register"/>
-        <state_interface name="latched_fault"/>
+        <state_interface name="error_code"/>
         <state_interface name="node_guard_error"/>
         <state_interface name="actual_motor_current"/>
-        <param name="can_id">22</param>
+        <param name="can_id">17</param>
         <param name="axis">1</param>
         <param name="path">"/home/rightbot/test_ws/src/ros2_control/rightbot_hardware_interface_pkgs/src/config/config.json"</param>
-        <param name="homing">1</param>
-        <param name="homing_at_zero">0</param>
-        <param name="homing_velocity">50</param>
-        <param name="homing_acceleration">10</param>
-        <param name="homing_position">0.951</param>
-        <param name="total_travel_distance">0.951</param>
-        <param name="motor_gear_ratio">7.5</param>
-        <param name="travel_per_revolution">0.314</param>
-        <param name="default_max_velocity">50.0</param>
-        <param name="default_max_accleration">10.0</param>
+        <param name="default_max_velocity">2</param>
+        <param name="default_max_accleration">0.5</param>
       </joint>
     </ros2_control>
-    <ros2_control name="TruckUnloading_rotation1_joint" type="actuator">
+     <ros2_control name="TruckUnloading_elbow_rotation_joint" type="actuator">
+      <hardware>
+        <plugin>harmonic_motor_actuator</plugin>
+        <param name="example_param_hw_start_duration_sec">0</param>
+        <param name="example_param_hw_stop_duration_sec">3.0</param>
+        <param name="example_param_hw_slowdown">100</param>
+      </hardware>
+      <joint name="elbow_rotation_joint">
+        <command_interface name="position">
+          <param name="min">-100</param>
+          <param name="max">100</param>
+        </command_interface>
+        <command_interface name="velocity"/>
+        <command_interface name="acceleration"/>
+        <state_interface name="position"/>
+        <state_interface name="velocity"/>
+        <state_interface name="status"/>
+        <state_interface name="error_code"/>
+        <state_interface name="node_guard_error"/>
+        <state_interface name="actual_motor_current"/>
+        <param name="can_id">18</param>
+        <param name="axis">-1</param>
+        <param name="path">"/home/rightbot/test_ws/src/ros2_control/rightbot_hardware_interface_pkgs/src/config/config.json"</param>
+        <param name="default_max_velocity">2</param>
+        <param name="default_max_accleration">0.5</param>
+      </joint>
+    </ros2_control>
+     <ros2_control name="TruckUnloading_wrist_rotation_joint" type="actuator">
+      <hardware>
+        <plugin>harmonic_motor_actuator</plugin>
+        <param name="example_param_hw_start_duration_sec">0</param>
+        <param name="example_param_hw_stop_duration_sec">3.0</param>
+        <param name="example_param_hw_slowdown">100</param>
+      </hardware>
+      <joint name="wrist_rotation_joint">
+        <command_interface name="position">
+          <param name="min">-100</param>
+          <param name="max">100</param>
+        </command_interface>
+        <command_interface name="velocity"/>
+        <command_interface name="acceleration"/>
+        <state_interface name="position"/>
+        <state_interface name="velocity"/>
+        <state_interface name="status"/>
+        <state_interface name="error_code"/>
+        <state_interface name="node_guard_error"/>
+        <state_interface name="actual_motor_current"/>
+        <param name="can_id">19</param>
+        <param name="axis">-1</param>
+        <param name="path">"/home/rightbot/test_ws/src/ros2_control/rightbot_hardware_interface_pkgs/src/config/config.json"</param>
+        <param name="default_max_velocity">4</param>
+        <param name="default_max_accleration">0.5</param>
+      </joint>
+    </ros2_control>
+     <ros2_control name="TruckUnloading_rotation1_joint" type="actuator">
       <hardware>
         <plugin>harmonic_motor_actuator</plugin>
@@ -63,6 +106,33 @@
         <param name="axis">-1</param>
         <param name="path">"/home/rightbot/test_ws/src/ros2_control/rightbot_hardware_interface_pkgs/src/config/config.json"</param>
-        <param name="default_max_velocity">2</param>
-        <param name="default_max_accleration">1</param>
+        <param name="default_max_velocity">4</param>
+        <param name="default_max_accleration">0.5</param>
+      </joint>
+    </ros2_control>
+     <ros2_control name="TruckUnloading_rotation2_joint" type="actuator">
+      <hardware>
+        <plugin>harmonic_motor_actuator</plugin>
+        <param name="example_param_hw_start_duration_sec">0</param>
+        <param name="example_param_hw_stop_duration_sec">3.0</param>
+        <param name="example_param_hw_slowdown">100</param>
+      </hardware>
+      <joint name="rotation2_joint">
+        <command_interface name="position">
+          <param name="min">-100</param>
+          <param name="max">100</param>
+        </command_interface>
+        <command_interface name="velocity"/>
+        <command_interface name="acceleration"/>
+        <state_interface name="position"/>
+        <state_interface name="velocity"/>
+        <state_interface name="status"/>
+        <state_interface name="error_code"/>
+        <state_interface name="node_guard_error"/>
+        <state_interface name="actual_motor_current"/>
+        <param name="can_id">21</param>
+        <param name="axis">-1</param>
+        <param name="path">"/home/rightbot/test_ws/src/ros2_control/rightbot_hardware_interface_pkgs/src/config/config.json"</param>
+        <param name="default_max_velocity">4</param>
+        <param name="default_max_accleration">0.5</param>
       </joint>
     </ros2_control>

Commit message: test launch file changes

File: rightbot_config_pkg/description/ros2_control/rightbot_test.ros2_control.xacro (robot description, xacro)
@@ -16,4 +16,5 @@
         <command_interface name="velocity"/>
         <command_interface name="acceleration"/>
+        <command_interface name="control_state"/>
         <state_interface name="position"/>
         <state_interface name="velocity"/>
@@ -21,5 +22,5 @@
         <state_interface name="error_code"/>
         <state_interface name="node_guard_error"/>
-        <state_interface name="actual_motor_current"/>
+        <state_interface name="effort"/>
         <param name="can_id">17</param>
         <param name="axis">1</param>
@@ -29,5 +30,5 @@
       </joint>
     </ros2_control>
-     <ros2_control name="TruckUnloading_elbow_rotation_joint" type="actuator">
+    <ros2_control name="TruckUnloading_elbow_rotation_joint" type="actuator">
       <hardware>
         <plugin>harmonic_motor_actuator</plugin>
@@ -43,4 +44,5 @@
         <command_interface name="velocity"/>
         <command_interface name="acceleration"/>
+        <command_interface name="control_state"/>
         <state_interface name="position"/>
         <state_interface name="velocity"/>
@@ -48,5 +50,5 @@
         <state_interface name="error_code"/>
         <state_interface name="node_guard_error"/>
-        <state_interface name="actual_motor_current"/>
+        <state_interface name="effort"/>
         <param name="can_id">18</param>
         <param name="axis">-1</param>
@@ -56,12 +58,9 @@
       </joint>
     </ros2_control>
-     <ros2_control name="TruckUnloading_wrist_rotation_joint" type="actuator">
+    <ros2_control name="TruckUnloading_camera_joint" type="actuator">
       <hardware>
-        <plugin>harmonic_motor_actuator</plugin>
-        <param name="example_param_hw_start_duration_sec">0</param>
-        <param name="example_param_hw_stop_duration_sec">3.0</param>
-        <param name="example_param_hw_slowdown">100</param>
+        <plugin>motor_actuator</plugin>
       </hardware>
-      <joint name="wrist_rotation_joint">
+      <joint name="camera_joint">
         <command_interface name="position">
           <param name="min">-100</param>
@@ -70,69 +69,22 @@
         <command_interface name="velocity"/>
         <command_interface name="acceleration"/>
+        <command_interface name="control_state"/>
+        <command_interface name="gpio"/>
         <state_interface name="position"/>
         <state_interface name="velocity"/>
         <state_interface name="status"/>
-        <state_interface name="error_code"/>
+        <state_interface name="battery_voltage"/>
+        <state_interface name="input_states"/>
+        <state_interface name="manufacturer_register"/>
+        <state_interface name="latched_fault"/>
         <state_interface name="node_guard_error"/>
-        <state_interface name="actual_motor_current"/>
-        <param name="can_id">19</param>
-        <param name="axis">-1</param>
+        <state_interface name="effort"/>
+        <param name="can_id">23</param>
+        <param name="axis">1</param>
         <param name="path">"/home/rightbot/test_ws/src/ros2_control/rightbot_hardware_interface_pkgs/src/config/config.json"</param>
-        <param name="default_max_velocity">4</param>
-        <param name="default_max_accleration">0.5</param>
-      </joint>
-    </ros2_control>
-     <ros2_control name="TruckUnloading_rotation1_joint" type="actuator">
-      <hardware>
-        <plugin>harmonic_motor_actuator</plugin>
-        <param name="example_param_hw_start_duration_sec">0</param>
-        <param name="example_param_hw_stop_duration_sec">3.0</param>
-        <param name="example_param_hw_slowdown">100</param>
-      </hardware>
-      <joint name="rotation1_joint">
-        <command_interface name="position">
-          <param name="min">-100</param>
-          <param name="max">100</param>
-        </command_interface>
-        <command_interface name="velocity"/>
-        <command_interface name="acceleration"/>
-        <state_interface name="position"/>
-        <state_interface name="velocity"/>
-        <state_interface name="status"/>
-        <state_interface name="error_code"/>
-        <state_interface name="node_guard_error"/>
-        <state_interface name="actual_motor_current"/>
-        <param name="can_id">20</param>
-        <param name="axis">-1</param>
-        <param name="path">"/home/rightbot/test_ws/src/ros2_control/rightbot_hardware_interface_pkgs/src/config/config.json"</param>
-        <param name="default_max_velocity">4</param>
-        <param name="default_max_accleration">0.5</param>
-      </joint>
-    </ros2_control>
-     <ros2_control name="TruckUnloading_rotation2_joint" type="actuator">
-      <hardware>
-        <plugin>harmonic_motor_actuator</plugin>
-        <param name="example_param_hw_start_duration_sec">0</param>
-        <param name="example_param_hw_stop_duration_sec">3.0</param>
-        <param name="example_param_hw_slowdown">100</param>
-      </hardware>
-      <joint name="rotation2_joint">
-        <command_interface name="position">
-          <param name="min">-100</param>
-          <param name="max">100</param>
-        </command_interface>
-        <command_interface name="velocity"/>
-        <command_interface name="acceleration"/>
-        <state_interface name="position"/>
-        <state_interface name="velocity"/>
-        <state_interface name="status"/>
-        <state_interface name="error_code"/>
-        <state_interface name="node_guard_error"/>
-        <state_interface name="actual_motor_current"/>
-        <param name="can_id">21</param>
-        <param name="axis">-1</param>
-        <param name="path">"/home/rightbot/test_ws/src/ros2_control/rightbot_hardware_interface_pkgs/src/config/config.json"</param>
-        <param name="default_max_velocity">4</param>
-        <param name="default_max_accleration">0.5</param>
+        <param name="homing">0</param>
+        <param name="motor_gear_ratio">7.5</param>
+        <param name="default_max_velocity">50.0</param>
+        <param name="default_max_accleration">10.0</param>
       </joint>
     </ros2_control>

Commit message: camera joint name changed to camera_rotation_joint

File: rightbot_config_pkg/description/ros2_control/rightbot_test.ros2_control.xacro (robot description, xacro)
@@ -58,9 +58,9 @@
       </joint>
     </ros2_control>
-    <ros2_control name="TruckUnloading_camera_joint" type="actuator">
+    <ros2_control name="TruckUnloading_camera_rotation_joint" type="actuator">
       <hardware>
         <plugin>motor_actuator</plugin>
       </hardware>
-      <joint name="camera_joint">
+      <joint name="camera_rotation_joint">
         <command_interface name="position">
           <param name="min">-100</param>

Commit message: underprogress

File: rightbot_config_pkg/description/ros2_control/rightbot_test.ros2_control.xacro (robot description, xacro)
@@ -2,12 +2,12 @@
 <robot xmlns:xacro="http://www.ros.org/wiki/xacro">
   <xacro:macro name="rightbot_test" params="name prefix slowdown:=2.0">
-    <ros2_control name="TruckUnloading_base_rotation_joint" type="actuator">
+    <ros2_control name="${name}_TruckUnloading_h_gantry_joint" type="actuator">
       <hardware>
-        <plugin>harmonic_motor_actuator</plugin>
+        <plugin>motor_actuator</plugin>
         <param name="example_param_hw_start_duration_sec">0</param>
         <param name="example_param_hw_stop_duration_sec">3.0</param>
         <param name="example_param_hw_slowdown">100</param>
       </hardware>
-      <joint name="base_rotation_joint">
+      <joint name="h_gantry_joint">
         <command_interface name="position">
           <param name="min">-100</param>
@@ -17,43 +17,29 @@
         <command_interface name="acceleration"/>
         <command_interface name="control_state"/>
+        <command_interface name="gpio"/>
         <state_interface name="position"/>
         <state_interface name="velocity"/>
         <state_interface name="status"/>
-        <state_interface name="error_code"/>
+        <state_interface name="battery_voltage"/>
+        <state_interface name="input_states"/>
+        <state_interface name="manufacturer_register"/>
+        <state_interface name="latched_fault"/>
         <state_interface name="node_guard_error"/>
         <state_interface name="effort"/>
-        <param name="can_id">17</param>
-        <param name="axis">1</param>
-        <param name="path">"/home/rightbot/test_ws/src/ros2_control/rightbot_hardware_interface_pkgs/src/config/config.json"</param>
-        <param name="default_max_velocity">2</param>
-        <param name="default_max_accleration">0.5</param>
-      </joint>
-    </ros2_control>
-    <ros2_control name="TruckUnloading_elbow_rotation_joint" type="actuator">
-      <hardware>
-        <plugin>harmonic_motor_actuator</plugin>
-        <param name="example_param_hw_start_duration_sec">0</param>
-        <param name="example_param_hw_stop_duration_sec">3.0</param>
-        <param name="example_param_hw_slowdown">100</param>
-      </hardware>
-      <joint name="elbow_rotation_joint">
-        <command_interface name="position">
-          <param name="min">-100</param>
-          <param name="max">100</param>
-        </command_interface>
-        <command_interface name="velocity"/>
-        <command_interface name="acceleration"/>
-        <command_interface name="control_state"/>
-        <state_interface name="position"/>
-        <state_interface name="velocity"/>
-        <state_interface name="status"/>
-        <state_interface name="error_code"/>
-        <state_interface name="node_guard_error"/>
-        <state_interface name="effort"/>
-        <param name="can_id">18</param>
+        <param name="can_id">16</param>
         <param name="axis">-1</param>
-        <param name="path">"/home/rightbot/test_ws/src/ros2_control/rightbot_hardware_interface_pkgs/src/config/config.json"</param>
-        <param name="default_max_velocity">2</param>
-        <param name="default_max_accleration">0.5</param>
+        <param name="path">
+          "/home/rightbot/test_ws/src/ros2_control/rightbot_hardware_interface_pkgs/src/config/config.json"
+        </param>
+        <param name="homing">1</param>
+        <param name="homing_at_zero">1</param>
+        <param name="homing_velocity">50</param>
+        <param name="homing_acceleration">10</param>
+        <param name="homing_position">0.709</param>
+        <param name="total_travel_distance">0.709</param>
+        <param name="motor_gear_ratio">1</param>
+        <param name="travel_per_revolution">0.032</param>
+        <param name="default_max_velocity">50.0</param>
+        <param name="default_max_accleration">25.0</param>
       </joint>
     </ros2_control>

Commit message: sending homing for camera if > 0.5 degree

File: rightbot_config_pkg/description/ros2_control/rightbot_test.ros2_control.xacro (robot description, xacro)
@@ -44,35 +44,4 @@
       </joint>
     </ros2_control>
-    <ros2_control name="TruckUnloading_camera_rotation_joint" type="actuator">
-      <hardware>
-        <plugin>motor_actuator</plugin>
-      </hardware>
-      <joint name="camera_rotation_joint">
-        <command_interface name="position">
-          <param name="min">-100</param>
-          <param name="max">100</param>
-        </command_interface>
-        <command_interface name="velocity"/>
-        <command_interface name="acceleration"/>
-        <command_interface name="control_state"/>
-        <command_interface name="gpio"/>
-        <state_interface name="position"/>
-        <state_interface name="velocity"/>
-        <state_interface name="status"/>
-        <state_interface name="battery_voltage"/>
-        <state_interface name="input_states"/>
-        <state_interface name="manufacturer_register"/>
-        <state_interface name="latched_fault"/>
-        <state_interface name="node_guard_error"/>
-        <state_interface name="effort"/>
-        <param name="can_id">23</param>
-        <param name="axis">1</param>
-        <param name="path">"/home/rightbot/test_ws/src/ros2_control/rightbot_hardware_interface_pkgs/src/config/config.json"</param>
-        <param name="homing">0</param>
-        <param name="motor_gear_ratio">7.5</param>
-        <param name="default_max_velocity">50.0</param>
-        <param name="default_max_accleration">10.0</param>
-      </joint>
-    </ros2_control>
     <ros2_control name="TruckUnloading_absolute_encoder_sensor" type="sensor">
       <hardware>
