Commit message: last working

File: rightbot_config_pkg/description/ros2_control/rightbot_test.ros2_control.xacro (robot description, xacro)
@@ -2,5 +2,5 @@
 <robot xmlns:xacro="http://www.ros.org/wiki/xacro">
   <xacro:macro name="rightbot_test" params="name prefix slowdown:=2.0">
-    <ros2_control name="${name}_TruckUnloading_h_gantry_joint" type="actuator">
+    <ros2_control name="${name}_TruckUnloading_v_gantry_joint" type="actuator">
       <hardware>
         <plugin>motor_actuator</plugin>
@@ -9,5 +9,5 @@
         <param name="example_param_hw_slowdown">100</param>
       </hardware>
-      <joint name="h_gantry_joint">
+      <joint name="v_gantry_joint">
         <command_interface name="position">
           <param name="min">-100</param>
@@ -27,19 +27,19 @@
         <state_interface name="node_guard_error"/>
         <state_interface name="effort"/>
-        <param name="can_id">16</param>
+        <param name="can_id">22</param>
         <param name="axis">-1</param>
+        <param name="homing">1</param>
+        <param name="homing_at_zero">0</param>
+        <param name="homing_velocity">50</param>
+        <param name="homing_acceleration">10</param>
+        <param name="homing_position">-0.951</param>
+        <param name="total_travel_distance">0.951</param>
+        <param name="motor_gear_ratio">7.5</param>
+        <param name="travel_per_revolution">0.314</param>
+        <param name="default_max_velocity">80.0</param>
+        <param name="default_max_accleration">25.0</param>
         <param name="path">
           "/home/rightbot/test_ws/src/ros2_control/rightbot_hardware_interface_pkgs/src/config/config.json"
         </param>
-        <param name="homing">1</param>
-        <param name="homing_at_zero">1</param>
-        <param name="homing_velocity">50</param>
-        <param name="homing_acceleration">10</param>
-        <param name="homing_position">0.709</param>
-        <param name="total_travel_distance">0.709</param>
-        <param name="motor_gear_ratio">1</param>
-        <param name="travel_per_revolution">0.032</param>
-        <param name="default_max_velocity">50.0</param>
-        <param name="default_max_accleration">25.0</param>
       </joint>
     </ros2_control>

Commit message: dummy actuator test

File: rightbot_config_pkg/description/ros2_control/rightbot_test.ros2_control.xacro (robot description, xacro)
@@ -2,5 +2,5 @@
 <robot xmlns:xacro="http://www.ros.org/wiki/xacro">
   <xacro:macro name="rightbot_test" params="name prefix slowdown:=2.0">
-    <ros2_control name="${name}_TruckUnloading_v_gantry_joint" type="actuator">
+    <!-- <ros2_control name="${name}_TruckUnloading_v_gantry_joint" type="actuator">
       <hardware>
         <plugin>motor_actuator</plugin>
@@ -43,6 +43,6 @@
         </param>
       </joint>
-    </ros2_control>
-    <ros2_control name="TruckUnloading_absolute_encoder_sensor" type="sensor">
+    </ros2_control> -->
+    <!-- <ros2_control name="TruckUnloading_absolute_encoder_sensor" type="sensor">
       <hardware>
         <plugin>absolute_encoder_sensor</plugin>
@@ -53,4 +53,60 @@
       <param name="axis">1</param>
     </sensor>
+    </ros2_control>  -->
+    <!-- <ros2_control name="${name}_TruckUnloading_rotation1_joint" type="actuator">
+      <hardware>
+        <plugin>harmonic_motor_actuator</plugin>
+        <param name="example_param_hw_start_duration_sec">0</param>
+        <param name="example_param_hw_stop_duration_sec">3.0</param>
+        <param name="example_param_hw_slowdown">100</param>
+      </hardware>
+      <joint name="rotation1_joint">
+        <command_interface name="position">
+          <param name="min">-100</param>
+          <param name="max">100</param>
+        </command_interface>
+        <command_interface name="velocity"/>
+        <command_interface name="acceleration"/>
+        <command_interface name="control_state"/>
+        <state_interface name="position"/>
+        <state_interface name="velocity"/>
+        <state_interface name="status"/>
+        <state_interface name="error_code"/>
+        <state_interface name="node_guard_error"/>
+        <state_interface name="effort"/>
+        <param name="can_id">20</param>
+        <param name="zero_point_count">0</param>
+        <param name="axis">1</param>
+        <param name="default_max_velocity">4</param>
+        <param name="default_max_accleration">0.5</param>
+        <param name="path">
+          "/home/rightbot/test_ws/src/ros2_control/rightbot_hardware_interface_pkgs/src/config/config.json"
+        </param>
+      </joint>
+    </ros2_control> -->
+    <ros2_control name="TruckUnloading_hinge_joint" type="actuator">
+      <hardware>
+        <plugin>dummy_actuator</plugin>
+        <param name="example_param_hw_start_duration_sec">0</param>
+        <param name="example_param_hw_stop_duration_sec">3.0</param>
+        <param name="example_param_hw_slowdown">100</param>
+      </hardware>
+      <joint name="hinge_joint">
+        <command_interface name="position">
+          <param name="min">-100</param>
+          <param name="max">100</param>
+        </command_interface>
+        <command_interface name="velocity"/>
+        <command_interface name="acceleration"/>
+        <command_interface name="control_state"/>
+        <state_interface name="position"/>
+        <state_interface name="velocity"/>
+        <state_interface name="status"/>
+        <state_interface name="error_code"/>
+        <state_interface name="node_guard_error"/>
+        <state_interface name="effort"/>
+        <param name="can_id">24</param>
+        <param name="axis">1</param>
+      </joint>
     </ros2_control>
   </xacro:macro>
