Commit message: SHER-784 Implement reinit function for STO recovery

File: rightbot_hardware_interface_pkgs/src/actuators/amc_motor_actuator_test/urdf/test.urdf (robot description, URDF)
Before this commit: robot test, 3 links, 2 joints
Joints:
- removed joint test_joint
- added joint conveyor_lift_left: type revolute, parent base_link, child link1, origin xyz=0 0 0.2 rpy=-1.57079632679 0 0, limit lower=-3.14159265359 upper=3.14159265359 effort=0.1 velocity=0.2

Commit message: Fix velocity command bug and rerun issue

File: rightbot_hardware_interface_pkgs/src/actuators/amc_motor_actuator_test/urdf/test.urdf (robot description, URDF)
Before this commit: robot test, 3 links, 2 joints
Joints:
- removed joint conveyor_lift_left
- added joint motor1: type revolute, parent base_link, child link1, origin xyz=0 0 0.2 rpy=-1.57079632679 0 0, limit lower=-3.14159265359 upper=3.14159265359 effort=0.1 velocity=0.2
